File: HW/SE/SE.kicad_pcb (KiCad board)
At the start: 2 copper layers, 59 parts, among them J1 Conn_01x03_Female, J2 Conn_01x07_Female, J3 Conn_01x02_Female, J4 Conn_01x02_Female, J5 Conn_01x02_Female, K1 SANYOU_SRD_Form_C, Q1 BSS138, Q2 BSS138, Q4 BC548, SW1 SW_Push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

Commit message: Inicio PCB
Parts:
- U2, U3: footprint Display:NHD-0420H1Z -> LIB:LCD_LCD-20X4B
- moved J2 175.8 mm to (20.0, 85.7)
- moved U4 174.0 mm to (40.7, 65.2)
- moved RV1 164.9 mm to (33.6, 53.0)
- moved Q2 154.6 mm to (66.2, 40.1)
- moved R4 152.1 mm to (54.6, 41.7)
- moved K1 141.8 mm to (30.1, 39.3)
- moved R1 134.2 mm to (57.2, 52.9)
- moved J1 130.5 mm to (43.4, 77.1)
- moved R6 122.9 mm to (66.1, 65.3)
- moved D3 121.6 mm to (79.2, 30.8)
- moved R5 118.9 mm to (76.7, 57.9)
- moved U3 117.1 mm to (163.7, 11.4)
- moved R11 112.0 mm to (100.0, 28.5)
- moved R3 111.8 mm to (67.9, 62.5)
- moved J3 109.2 mm to (120.2, 142.7), turned to 90 degrees
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Connections:
- net MISO renamed Net-(J2-Pad4)
- net MOSI renamed Net-(J2-Pad3)
- net RST renamed Net-(J2-Pad6)
- net SCKs renamed Net-(J2-Pad2)
- net SDAs renamed Net-(J2-Pad1)
- R10 pad 2: 3.33v -> +3V3
- R9 pad 2: 3.33v -> +3V3

Commit message: A
Parts:
- moved J1 224.5 mm to (267.1, 59.3)
- moved J2 195.7 mm to (210.5, 41.2)
- moved U4 143.2 mm to (176.8, 109.8)
- moved K1 142.8 mm to (144.3, 125.1), turned to 180 degrees
- moved SW3 119.1 mm to (267.7, 84.0)
- moved C3 119.1 mm to (252.2, 94.0)
- moved SW1 119.1 mm to (261.1, 86.4)
- moved SW2 119.1 mm to (253.9, 82.8)
- moved C2 119.1 mm to (262.0, 94.9)
- moved R4 104.5 mm to (135.6, 107.8)
- moved RV1 103.9 mm to (132.4, 85.4)
- moved R3 98.4 mm to (158.5, 101.0)
- moved R5 98.4 mm to (167.2, 96.4)
- moved R6 98.4 mm to (156.6, 103.8)
- moved R14 97.5 mm to (163.0, 124.3), turned to 180 degrees
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
Commit message: Ajuste PCB
Parts:
- moved U2 122.9 mm to (143.8, 105.0)
- moved J1 99.6 mm to (207.7, 139.1), turned to 180 degrees
- moved U3 86.6 mm to (143.9, 95.8)
- moved R4 75.8 mm to (199.7, 67.3)
- moved C1 45.7 mm to (121.9, 37.2)
- moved D2 45.7 mm to (136.6, 34.3)
- moved Q1 45.7 mm to (172.2, 56.2)
- moved R12 45.7 mm to (167.6, 54.6)
- moved R13 45.7 mm to (131.2, 51.3)
- moved R9 45.7 mm to (145.4, 51.3)
- moved D3 45.7 mm to (124.9, 29.2)
- moved Q2 45.7 mm to (111.9, 38.5)
- moved R1 45.7 mm to (102.9, 51.3)
- moved R10 45.7 mm to (149.4, 51.3)
- moved R11 45.7 mm to (145.7, 26.9)
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
Commit message: Distribucion final de componetes en 10*10
Parts:
- SW1: value SW_Push -> Program
- moved Q2 107.4 mm to (175.1, 125.4), turned to 90 degrees
- moved D3 103.1 mm to (175.2, 119.2)
- moved R11 93.9 mm to (182.7, 113.3)
- moved D2 87.9 mm to (175.1, 113.3)
- moved R9 87.2 mm to (180.6, 131.1), turned to 270 degrees
- moved R1 84.6 mm to (185.5, 69.3)
- moved R10 80.5 mm to (180.6, 125.5), turned to 270 degrees
- moved C1 79.6 mm to (192.1, 74.7)
- moved D1 78.1 mm to (175.2, 107.4)
- moved Q1 75.0 mm to (175.0, 131.1), turned to 90 degrees
- moved SW1 70.3 mm to (199.6, 68.4), turned to 0 degrees
- moved R12 66.3 mm to (182.7, 119.2)
- moved R4 65.4 mm to (169.5, 125.4), turned to 90 degrees
- moved R2 62.4 mm to (182.7, 107.4)
- moved SW3 61.3 mm to (208.3, 68.8), turned to 180 degrees
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