File: HW/SE/SE.kicad_pcb (KiCad board)
At the start: 2 copper layers, 59 parts, among them J1 Conn_01x03_Female, J2 Conn_01x07_Female, J3 Conn_01x02_Female, J4 Conn_01x02_Female, J5 Conn_01x02_Female, K1 SANYOU_SRD_Form_C, Q1 BSS138, Q2 BSS138, Q4 BC548, SW1 Program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

Commit message: Conecciones Iniciales
Routing:
- net Net-(D6-Pad1): track 0.00 -> 18.8 mm
- net +12V: track 0.00 -> 18.3 mm
- net Net-(D6-Pad2): track 0.00 -> 16.5 mm
- net Vbat: track 0.00 -> 5.63 mm
- net Net-(F1-Pad1): track 0.00 -> 5.50 mm
Changed lines of the file:
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@@
     (thickness 1.6)
     (drawings 4)
-    (tracks 0)
+    (tracks 23)
     (zones 0)
     (modules 59)
@@
     (via_min_size 0.4)
     (via_min_drill 0.3)
+    (user_via 0.525491 0.3)
     (uvia_size 0.3)
     (uvia_drill 0.1)
@@
     (arrow2b (pts (xy 111.79 157.63) (xy 112.916504 157.043579)))
   )
+  (segment (start 145.13 143.205) (end 151.18 143.205) (width 0.525491) (layer F.Cu) (net 6))
+  (segment (start 151.905 143.93) (end 151.18 143.205) (width 0.525491) (layer F.Cu) (net 6))
+  (segment (start 156.37 143.93) (end 151.905 143.93) (width 0.525491) (layer F.Cu) (net 6))
+  (segment (start 139.145 143.205) (end 138.63 143.72) (width 0.525491) (layer F.Cu) (net 6))
+  (segment (start 145.13 143.205) (end 139.145 143.205) (width 0.525491) (layer F.Cu) (net 6))
+  (segment (start 134.2175 129.29) (end 135.7575 130.83) (width 0.525491) (layer F.Cu) (net 13))
+  (segment (start 130.325 129.29) (end 134.2175 129.29) (width 0.525491) (layer F.Cu) (net 13))
+  (segment (start 135.745 130.8425) (end 135.7575 130.83) (width 0.525491) (layer F.Cu) (net 13))
+  (segment (start 135.745 134.98) (end 135.745 130.8425) (width 0.525491) (layer F.Cu) (net 13))
+  (segment (start 135.355 135.37) (end 135.745 134.98) (width 0.525491) (layer F.Cu) (net 13))
+  (segment (start 129.61 135.37) (end 135.355 135.37) (width 0.525491) (layer F.Cu) (net 13))
+  (segment (start 126.81 135.37) (end 126.81 139.25) (width 0.525491) (layer F.Cu) (net 14))
+  (segment (start 128.136 140.576) (end 128.136 142.8548) (width 0.525491) (layer F.Cu) (net 14))
+  (segment (start 126.81 139.25) (end 128.136 140.576) (width 0.525491) (layer F.Cu) (net 14))
+  (segment (start 128.136 142.8548) (end 129.7652 142.8548) (width 0.525491) (layer F.Cu) (net 14))
+  (segment (start 129.7652 142.8548) (end 131.43 141.19) (width 0.525491) (layer F.Cu) (net 14))
+  (segment (start 136.13 141.944509) (end 136.13 143.72) (width 0.525491) (layer F.Cu) (net 14))
+  (segment (start 135.375491 141.19) (end 136.13 141.944509) (width 0.525491) (layer F.Cu) (net 14))
+  (segment (start 131.43 141.19) (end 135.375491 141.19) (width 0.525491) (layer F.Cu) (net 14))
+  (segment (start 125.855 129.31) (end 125.875 129.29) (width 0.525491) (layer F.Cu) (net 17))
+  (segment (start 120.38 129.31) (end 125.855 129.31) (width 0.525491) (layer F.Cu) (net 17))
+  (segment (start 126.054 143.77) (end 126.104 143.82) (width 0.525491) (layer F.Cu) (net 20))
+  (segment (start 120.49 143.77) (end 126.054 143.77) (width 0.525491) (layer F.Cu) (net 20))
 )

Commit message: Ruteo y dimensionamiento
Parts:
- added REF**: MountingHole_2.2mm_M2_ISO14580_Pad, MountingHole:MountingHole_2.2mm_M2_ISO14580_Pad, F.Cu at (207.7, 147.9)
- added REF**: MountingHole_2.2mm_M2_ISO14580_Pad, MountingHole:MountingHole_2.2mm_M2_ISO14580_Pad, F.Cu at (207.7, 61.8)
- added REF**: MountingHole_2.2mm_M2_ISO14580_Pad, MountingHole:MountingHole_2.2mm_M2_ISO14580_Pad, F.Cu at (115.7, 61.8)
- moved D7 30.5 mm to (145.5, 133.1), turned to 180 degrees
- moved D8 30.1 mm to (145.3, 127.0), turned to 180 degrees
- moved R7 11.7 mm to (162.2, 102.2), turned to 0 degrees
- moved R6 5.92 mm to (162.2, 97.9), turned to 0 degrees
- moved R8 5.34 mm to (154.4, 93.5), turned to 0 degrees
- moved J1 3.46 mm to (200.5, 133.2)
- moved R5 2.45 mm to (162.1, 93.8), turned to 0 degrees
Routing:
- net +5V: track 0.00 -> 224.0 mm, vias 0 -> 2
- net +3V3: track 0.00 -> 181.6 mm, vias 0 -> 2
- net Net-(Q2-Pad3): track 0.00 -> 72.2 mm, vias 0 -> 3
- net Net-(U2-Pad6): track 0.00 -> 70.0 mm, vias 0 -> 2
- net Net-(U2-Pad5): track 0.00 -> 67.0 mm, vias 0 -> 2
- net Net-(U2-Pad4): track 0.00 -> 62.5 mm, vias 0 -> 2
- net Net-(R12-Pad2): track 0.00 -> 58.7 mm, vias 0 -> 2
- net Crelay: track 0.00 -> 55.7 mm, vias 0 -> 2
- net Net-(C3-Pad2): track 0.00 -> 55.6 mm, vias 0 -> 3
- net SCL: track 0.00 -> 52.9 mm, vias 0 -> 2
- net Net-(R11-Pad2): track 0.00 -> 51.3 mm, vias 0 -> 2
- net Net-(U2-Pad11): track 0.00 -> 46.4 mm
- net SDA: track 0.00 -> 43.5 mm
- net Net-(J2-Pad2): track 0.00 -> 42.8 mm, vias 0 -> 1
- net Net-(U2-Pad12): track 0.00 -> 42.2 mm
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Other:
- board outline added: 100.2 x 94.3 mm

Commit message: PCB lista
Parts:
- added REF**: MountingHole_2.2mm_M2_ISO14580_Pad, MountingHole:MountingHole_2.2mm_M2_ISO14580_Pad, F.Cu at (115.7, 147.9)
- moved J4 3.14 mm to (120.1, 140.7)
Routing:
- net Net-(Q1-Pad3): track 11.2 -> 83.0 mm
- net Vbat: track 5.63 -> 7.95 mm
- added copper zone on B.Cu, net (none)
- added copper zone on F.Cu, net GND
Other:
- board size 100.2 x 94.3 mm -> 100.1 x 94.1 mm
Changed lines of the file:
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@@
   (general
     (thickness 1.6)
-    (drawings 7)
-    (tracks 456)
+    (drawings 6)
+    (tracks 470)
     (zones 0)
-    (modules 62)
+    (modules 63)
     (nets 78)
   )
@@
   )
   (module MountingHole:MountingHole_2.2mm_M2_ISO14580_Pad (layer F.Cu)
+    (at 115.65 147.87)
+    (descr "Mounting Hole 2.2mm, M2, ISO14580")
+    (tags "mounting hole 2.2mm m2 iso14580")
+    (attr virtual)
+    (fp_text reference REF** (at 0 -2.9) (layer F.SilkS)
+      (effects (font (size 1 1) (thickness 0.15)))
+    )
+    (fp_text value MountingHole_2.2mm_M2_ISO14580_Pad (at 0 2.9) (layer F.Fab)
+      (effects (font (size 1 1) (thickness 0.15)))
+    )
+    (fp_text user %R (at 0.3 0) (layer F.Fab)
+      (effects (font (size 1 1) (thickness 0.15)))
+    )
+    (fp_circle (center 0 0) (end 2.15 0) (layer F.CrtYd) (width 0.05))
+    (fp_circle (center 0 0) (end 1.9 0) (layer Cmts.User) (width 0.15))
+    (pad 1 thru_hole circle (at 0 0) (size 3.8 3.8) (drill 2.2) (layers *.Cu *.Mask))
+  )
+  (module MountingHole:MountingHole_2.2mm_M2_ISO14580_Pad (layer F.Cu)
     (at 207.67 147.95)
     (descr "Mounting Hole 2.2mm, M2, ISO14580")
@@
   )
   (module Connector_Molex:Molex_Micro-Latch_53254-0270_1x02_P2.00mm_Horizontal (layer F.Cu)
-    (at 120.49 143.77 90)
+    (at 120.07 140.66 90)
     (descr "Molex Micro-Latch Wire-to-Board Connector System, 53254-0270 (compatible alternatives: 53254-0250), 2 Pins per row (http://www.molex.com/pdm_docs/sd/532530770_sd.pdf), generated with kicad-footprint-generator")
     (tags "connector Molex Micro-Latch top entry")
@@
     )
   )
+  (gr_line (start 211.72 151.85) (end 211.65 57.83) (layer Edge.Cuts) (width 0.1))
+  (gr_line (start 111.73 151.93) (end 211.72 151.85) (layer Edge.Cuts) (width 0.1))
+  (gr_line (start 111.62 57.89) (end 111.73 151.93) (layer Edge.Cuts) (width 0.1))
+  (gr_line (start 211.65 57.83) (end 111.62 57.89) (layer Edge.Cuts) (width 0.1))
   (dimension 94.000043 (width 0.15) (layer Dwgs.User)
-    (gr_text "94.000 mm" (at 217.944812 104.854006 -89.94514236) (layer Dwgs.User)
+    (gr_text "94.000 mm" (at 107.165 104.960073 -89.94514236) (layer Dwgs.User)
       (effects (font (size 1 1) (thickness 0.15)))
     )
-    (feature1 (pts (xy 211.64 57.86) (xy 217.186233 57.85469)))
-    (feature2 (pts (xy 211.73 151.86) (xy 217.276233 151.85469)))
-    (crossbar (pts (xy 216.689813 151.855251) (xy 216.599813 57.855251)))
-    (arrow1a (pts (xy 216.599813 57.855251) (xy 217.187312 58.981193)))
-    (arrow1b (pts (xy 216.599813 57.855251) (xy 216.014471 58.982316)))
-    (arrow2a (pts (xy 216.689813 151.855251) (xy 217.275155 150.728186)))
-    (arrow2b (pts (xy 216.689813 151.855251) (xy 216.102314 150.729309)))
+    (feature1 (pts (xy 211.64 57.86) (xy 107.833579 57.959389)))
+    (feature2 (pts (xy 211.73 151.86) (xy 107.923579 151.959389)))
+    (crossbar (pts (xy 108.509999 151.958828) (xy 108.419999 57.958828)))
+    (arrow1a (pts (xy 108.419999 57.958828) (xy 109.007498 59.08477)))
+    (arrow1b (pts (xy 108.419999 57.958828) (xy 107.834657 59.085893)))
+    (arrow2a (pts (xy 108.509999 151.958828) (xy 109.095341 150.831763)))
+    (arrow2b (pts (xy 108.509999 151.958828) (xy 107.9225 150.832886)))
   )
   (dimension 100.040072 (width 0.15) (layer Dwgs.User)
-    (gr_text "100.040 mm" (at 161.75379 155.080008 0.06872741148) (layer Dwgs.User)
+    (gr_text "100.040 mm" (at 161.631128 52.819998 0.06872741148) (layer Dwgs.User)
       (effects (font (size 1 1) (thickness 0.15)))
     )
-    (feature1 (pts (xy 211.77 151.86) (xy 211.772935 154.306429)))
-    (feature2 (pts (xy 111.73 151.98) (xy 111.732935 154.426429)))
-    (crossbar (pts (xy 111.732231 153.840009) (xy 211.772231 153.720009)))
-    (arrow1a (pts (xy 211.772231 153.720009) (xy 210.646431 154.307781)))
-    (arrow1b (pts (xy 211.772231 153.720009) (xy 210.645025 153.13494)))
-    (arrow2a (pts (xy 111.732231 153.840009) (xy 112.859437 154.425078)))
-    (arrow2b (pts (xy 111.732231 153.840009) (xy 112.858031 153.252237)))
-  )
-  (gr_line (start 111.74 152) (end 111.95 151.98) (layer Edge.Cuts) (width 0.1))
-  (gr_line (start 111.61 57.69) (end 111.74 152) (layer Edge.Cuts) (width 0.1))
-  (gr_line (start 211.63 57.82) (end 111.61 57.69) (layer Edge.Cuts) (width 0.1))
-  (gr_line (start 211.77 151.85) (end 211.63 57.82) (layer Edge.Cuts) (width 0.1))
-  (gr_line (start 111.96 151.98) (end 211.77 151.85) (layer Edge.Cuts) (width 0.1))
+    (feature1 (pts (xy 211.77 151.86) (xy 211.651983 53.473577)))
+    (feature2 (pts (xy 111.73 151.98) (xy 111.611983 53.593577)))
+    (crossbar (pts (xy 111.612687 54.179997) (xy 211.652687 54.059997)))
+    (arrow1a (pts (xy 211.652687 54.059997) (xy 210.526887 54.647769)))
+    (arrow1b (pts (xy 211.652687 54.059997) (xy 210.525481 53.474928)))
+    (arrow2a (pts (xy 111.612687 54.179997) (xy 112.739893 54.765066)))
+    (arrow2b (pts (xy 111.612687 54.179997) (xy 112.738487 53.592225)))
+  )
   (via (at 200.65 124.93) (size 0.8) (drill 0.4) (layers F.Cu B.Cu) (net 24))
   (via (at 180.61 128.41) (size 0.8) (drill 0.4) (layers F.Cu B.Cu) (net 24))
@@
   (segment (start 167.24125 128.59125) (end 169.54 126.2925) (width 0.25) (layer F.Cu) (net 7))
   (segment (start 167.1 128.7325) (end 167.24125 128.59125) (width 0.25) (layer F.Cu) (net 7))
-  (segment (start 162.67 136.82) (end 162.76 136.73) (width 0.25) (layer F.Cu) (net 7))
   (segment (start 125.75 88.32) (end 125.73 88.34) (width 0.25) (layer B.Cu) (net 7))
   (segment (start 125.75 79.16) (end 125.75 88.32) (width 0.25) (layer B.Cu) (net 7))
@@
   (segment (start 195.01 132.65) (end 195.58 133.22) (width 0.25) (layer F.Cu) (net 19))
   (segment (start 126.054 143.77) (end 126.104 143.82) (width 0.525491) (layer F.Cu) (net 20))
-  (segment (start 120.49 143.77) (end 126.054 143.77) (width 0.525491) (layer F.Cu) (net 20))
+  (segment (start 126.104 143.82) (end 125.49 143.82) (width 0.525491) (layer F.Cu) (net 20))
+  (segment (start 125.49 143.82) (end 123.67 142) (width 0.525491) (layer F.Cu) (net 20))
+  (segment (start 123.67 142) (end 123.67 141.09) (width 0.525491) (layer F.Cu) (net 20))
+  (segment (start 123.24 140.66) (end 120.07 140.66) (width 0.525491) (layer F.Cu) (net 20))
+  (segment (start 123.67 141.09) (end 123.24 140.66) (width 0.525491) (layer F.Cu) (net 20))
   (segment (start 120.4 107.49) (end 122.63 107.49) (width 0.525491) (layer F.Cu) (net 21))
   (segment (start 128.66 113.52) (end 144.53 113.52) (width 0.525491) (layer F.Cu) (net 21))
@@
   (segment (start 169.6 128.53) (end 169.54 128.59) (width 0.25) (layer B.Cu) (net 23))
   (segment (start 175.02 128.53) (end 169.6 128.53) (width 0.25) (layer B.Cu) (net 23))
+  (segment (start 169.73 76.83) (end 169.73 75.91) (width 0.25) (layer B.Cu) (net 23))
+  (segment (start 169.73 75.91) (end 170.4 75.24) (width 0.25) (layer B.Cu) (net 23))
+  (segment (start 170.4 75.24) (end 175.5 75.24) (width 0.25) (layer B.Cu) (net 23))
+  (segment (start 175.5 75.24) (end 176.8 76.54) (width 0.25) (layer B.Cu) (net 23))
+  (segment (start 176.8 76.54) (end 176.8 120.59) (width 0.25) (layer B.Cu) (net 23))
+  (segment (start 176.8 120.59) (end 176.11 121.28) (width 0.25) (layer B.Cu) (net 23))
+  (segment (start 176.11 121.28) (end 168.34 121.28) (width 0.25) (layer B.Cu) (net 23))
+  (segment (start 168.34 121.28) (end 166.66 122.96) (width 0.25) (layer B.Cu) (net 23))
+  (segment (start 166.66 122.96) (end 166.66 127.47) (width 0.25) (layer B.Cu) (net 23))
+  (segment (start 167.78 128.59) (end 169.54 128.59) (width 0.25) (layer B.Cu) (net 23))
+  (segment (start 166.66 127.47) (end 167.78 128.59) (width 0.25) (layer B.Cu) (net 23))
   (segment (start 175.97 132.11) (end 177.29 132.11) (width 0.25) (layer F.Cu) (net 24))
   (segment (start 179.2225 130.1775) (end 180.59 130.1775) (width 0.25) (layer F.Cu) (net 24))
@@
   (segment (start 199.08 103.9) (end 192.29 103.9) (width 0.25) (layer B.Cu) (net 77))
   (segment (start 203.82 108.64) (end 199.08 103.9) (width 0.25) (layer B.Cu) (net 77))
+  (zone (net 1) (net_name GND) (layer F.Cu) (hatch edge 0.508)
+    (connect_pads (clearance 0.508))
+    (min_thickness 0.254)
+    (fill yes (arc_segments 32) (thermal_gap 0.508) (thermal_bridge_width 0.508))
+    (polygon
+      (pts
+        (xy 212.91 153.65) (xy 110.04 154.33) (xy 110.45 57.21) (xy 110.75 57.27) (xy 213.04 57)
+      )
+    )
+  )
+  (zone (net 0) (net_name "") (layer B.Cu) (hatch edge 0.508)
+    (connect_pads (clearance 0.508))
+    (min_thickness 0.254)
+    (fill yes (arc_segments 32) (thermal_gap 0.508) (thermal_bridge_width 0.508))
+    (polygon
+      (pts
+        (xy 213.67 56.77) (xy 214.48 155.8) (xy 107.42 155.8) (xy 108.5 56.9) (xy 109.95 56.73)
+      )
+    )
+  )
 )

Commit message: Nombramiento puertos y testigos
Other:
- board text added: "+"
- board text added: "-"
- board text added: "A"
- board text added: "BATERIA"
- board text added: "DB0"
- board text added: "DB1"
- board text added: "DB2"
- board text added: "DB3"
- board text added: "DB4"
- board text added: "DB5"
- board text added: "DB6"
- board text added: "DB7"
- board text added: "E"
- board text added: "Encendido"
- board text added: "FUENTE"
- board text added: "Fuente"
- board text added: "GND"
- board text added: "IMAN"
- board text added: "K"
- board text added: "MISO"
- board text added: "MOSI"
- board text added: "Program"
- board text added: "Puerta"
- board text added: "R/W"
- board text added: "RS"
- board text added: "RST"
- board text added: "RX"
- board text added: "Reset"
- board text added: "ResetP"
- board text added: "SCK"
- board text added: "SDA"
- board text added: "TX"
- board text added: "VDD"
- board text added: "VSS"
- board text added: "Vcc"
- board text added: "Vo"
Changed lines of the file:
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@@
   (general
     (thickness 1.6)
-    (drawings 6)
+    (drawings 45)
     (tracks 470)
     (zones 0)
@@
   (module LIB:LCD_LCD-20X4B (layer F.Cu)
     (at 143.16 78.68)
-    (fp_text reference U3 (at -0.6 3.39) (layer F.SilkS)
+    (fp_text reference U3 (at -0.29 -1.95) (layer F.SilkS)
       (effects (font (size 1.4 1.4) (thickness 0.15)))
     )
@@
     )
   )
+  (gr_text Program (at 191.79 70.37) (layer F.SilkS)
+    (effects (font (size 1 1) (thickness 0.15)))
+  )
+  (gr_text ResetP (at 199.76 70.75) (layer F.SilkS)
+    (effects (font (size 1 1) (thickness 0.15)))
+  )
+  (gr_text Reset (at 208.17 66.29) (layer F.SilkS)
+    (effects (font (size 1 1) (thickness 0.15)))
+  )
+  (gr_text Puerta (at 153.55 110.47) (layer F.SilkS)
+    (effects (font (size 1 1) (thickness 0.15)))
+  )
+  (gr_text Encendido (at 145.15 124.52) (layer F.SilkS)
+    (effects (font (size 1 1) (thickness 0.15)))
+  )
+  (gr_text Fuente (at 145.62 130.7) (layer F.SilkS)
+    (effects (font (size 1 1) (thickness 0.15)))
+  )
+  (gr_text IMAN (at 116.01 102.34) (layer F.SilkS)
+    (effects (font (size 1 1) (thickness 0.15)))
+  )
+  (gr_text - (at 122.55 138.94) (layer F.SilkS)
+    (effects (font (size 1 1) (thickness 0.15)))
+  )
+  (gr_text - (at 122.64 127.5) (layer F.SilkS)
+    (effects (font (size 1 1) (thickness 0.15)))
+  )
+  (gr_text + (at 122.36 129.1) (layer F.SilkS)
+    (effects (font (size 1 1) (thickness 0.15)))
+  )
+  (gr_text + (at 122.27 140.63) (layer F.SilkS)
+    (effects (font (size 1 1) (thickness 0.15)))
+  )
+  (gr_text BATERIA (at 116.64 135.56) (layer F.SilkS)
+    (effects (font (size 1 1) (thickness 0.15)))
+  )
+  (gr_text FUENTE (at 117.58 124.13) (layer F.SilkS)
+    (effects (font (size 1 1) (thickness 0.15)))
+  )
+  (gr_text K (at 161.34 86.06 90) (layer F.SilkS)
+    (effects (font (size 1 1) (thickness 0.15)))
+  )
+  (gr_text A (at 158.71 85.97 90) (layer F.SilkS)
+    (effects (font (size 1 1) (thickness 0.15)))
+  )
+  (gr_text DB7 (at 156.37 85.4 90) (layer F.SilkS)
+    (effects (font (size 1 1) (thickness 0.15)))
+  )
+  (gr_text DB6 (at 153.74 85.5 90) (layer F.SilkS)
+    (effects (font (size 1 1) (thickness 0.15)))
+  )
+  (gr_text DB5 (at 151.31 85.4 90) (layer F.SilkS)
+    (effects (font (size 1 1) (thickness 0.15)))
+  )
+  (gr_text DB4 (at 148.78 85.5 90) (layer F.SilkS)
+    (effects (font (size 1 1) (thickness 0.15)))
+  )
+  (gr_text DB3 (at 146.15 85.55 90) (layer F.SilkS)
+    (effects (font (size 1 1) (thickness 0.15)))
+  )
+  (gr_text DB2 (at 143.62 85.55 90) (layer F.SilkS)
+    (effects (font (size 1 1) (thickness 0.15)))
+  )
+  (gr_text DB1 (at 140.9 85.55 90) (layer F.SilkS)
+    (effects (font (size 1 1) (thickness 0.15)))
+  )
+  (gr_text DB0 (at 138.46 85.64 90) (layer F.SilkS)
+    (effects (font (size 1 1) (thickness 0.15)))
+  )
+  (gr_text E (at 136.12 86.2 90) (layer F.SilkS)
+    (effects (font (size 1 1) (thickness 0.15)))
+  )
+  (gr_text R/W (at 133.4 85.45 90) (layer F.SilkS)
+    (effects (font (size 1 1) (thickness 0.15)))
+  )
+  (gr_text RS (at 130.78 85.83 90) (layer F.SilkS)
+    (effects (font (size 1 1) (thickness 0.15)))
+  )
+  (gr_text Vo (at 128.34 85.83 90) (layer F.SilkS)
+    (effects (font (size 1 1) (thickness 0.15)))
+  )
+  (gr_text VSS (at 123.28 85.45 90) (layer F.SilkS)
+    (effects (font (size 1 1) (thickness 0.15)))
+  )
+  (gr_text VDD (at 125.81 85.45 90) (layer F.SilkS)
+    (effects (font (size 1 1) (thickness 0.15)))
+  )
+  (gr_text RX (at 198.08 130.73) (layer F.SilkS)
+    (effects (font (size 1 1) (thickness 0.15)))
+  )
+  (gr_text TX (at 198.03 133.27) (layer F.SilkS)
+    (effects (font (size 1 1) (thickness 0.15)))
+  )
+  (gr_text GND (at 197.8 128.13) (layer F.SilkS)
+    (effects (font (size 1 1) (thickness 0.15)))
+  )
+  (gr_text "Vcc\n" (at 200.81 122.12) (layer F.SilkS)
+    (effects (font (size 1 1) (thickness 0.15)))
+  )
+  (gr_text RST (at 200.63 120.3) (layer F.SilkS)
+    (effects (font (size 1 1) (thickness 0.15)))
+  )
+  (gr_text GND (at 200.72 118.34) (layer F.SilkS)
+    (effects (font (size 1 1) (thickness 0.15)))
+  )
+  (gr_text MISO (at 200.54 116.32) (layer F.SilkS)
+    (effects (font (size 1 1) (thickness 0.15)))
+  )
+  (gr_text MOSI (at 200.57 114.32) (layer F.SilkS)
+    (effects (font (size 1 1) (thickness 0.15)))
+  )
+  (gr_text "SCK\n" (at 200.66 112.24) (layer F.SilkS)
+    (effects (font (size 1 1) (thickness 0.15)))
+  )
+  (gr_text "SDA\n" (at 200.58 110.19) (layer F.SilkS)
+    (effects (font (size 1 1) (thickness 0.15)))
+  )
   (gr_line (start 211.72 151.85) (end 211.65 57.83) (layer Edge.Cuts) (width 0.1))

Commit message: Ajustes Finales PCB
Parts:
- C1, C10, C2, C3, C4, C5, C6, C7, C8, C9: footprint Capacitor_SMD:C_1210_3225Metric_Pad1.33x2.70mm_HandSolder -> Capacitor_SMD:C_1206_3216Metric_Pad1.33x1.80mm_HandSolder
- D1, D2, D3, D4, D7, D8: footprint LED_SMD:LED_1210_3225Metric_Pad1.42x2.65mm_HandSolder -> LED_SMD:LED_0805_2012Metric_Pad1.15x1.40mm_HandSolder
- moved C7 6.12 mm to (181.1, 141.8)
- moved C4 5.81 mm to (150.9, 141.9)
- moved C5 5.74 mm to (145.5, 142.1)
- moved C8 5.70 mm to (175.2, 141.9)
- moved D1 2.00 mm to (173.2, 107.4)
- moved D3 1.96 mm to (173.3, 119.1)
- moved D2 1.88 mm to (173.3, 113.3)
- moved C9 0.95 mm to (199.0, 141.5)
- moved C10 0.84 mm to (204.2, 141.6)
- moved C6 0.67 mm to (169.5, 141.9)
- moved C2 0.59 mm to (208.1, 74.3)
- moved C1 0.33 mm to (192.2, 75.0)
- moved C3 0.28 mm to (199.4, 74.8)
- moved D8 0.18 mm to (145.4, 127.0)
- moved D7 0.15 mm to (145.4, 133.2)
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Routing:
- net Net-(D1-Pad2): track 5.17 -> 7.63 mm
- net Net-(D3-Pad2): track 5.10 -> 7.53 mm
- net Net-(D2-Pad2): track 5.12 -> 7.47 mm
- net +3V3: track 181.6 -> 183.3 mm
- net Net-(C2-Pad2): track 20.2 -> 21.7 mm
- net +5V: track 223.9 -> 225.0 mm
- net Net-(C1-Pad1): track 29.8 -> 30.5 mm
- net Net-(D8-Pad2): track 6.41 -> 7.05 mm
- added copper zone on B.Cu, net GND
- removed copper zone on B.Cu, net (none)
Other:
- board text added: "Error"
- board text added: "OK"
- board text removed: "ResetP"
