File: HW/SE/SE.sch (KiCad schematic (older format))
At the start: 57 parts, among them J1 Conn_01x03_Female, J2 Conn_01x07_Female, J3 Conn_01x02_Female, J4 Conn_01x02_Female, J5 Conn_01x02_Female, K1 SANYOU_SRD_Form_C, Q1 BSS138, Q2 BSS138, Q4 BC548, SW1 SW_Push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

Commit message: A
Parts:
- SW1, SW2, SW3: footprint (none) -> Button_Switch_SMD:SW_Push_SPST_NO_Alps_SKRK
- SW4: footprint (none) -> Button_Switch_SMD:SW_SPDT_CK-JS102011SAQN
Changed lines of the file:
@@
 F 0 "SW1" H 4050 1535 50  0000 C CNN
 F 1 "SW_Push" H 4050 1444 50  0000 C CNN
-F 2 "" H 4050 1450 50  0001 C CNN
+F 2 "Button_Switch_SMD:SW_Push_SPST_NO_Alps_SKRK" H 4050 1450 50  0001 C CNN
 F 3 "~" H 4050 1450 50  0001 C CNN
 	1    4050 1250
@@
 F 0 "SW2" H 1400 2085 50  0000 C CNN
 F 1 "ResetP" H 1400 1994 50  0000 C CNN
-F 2 "" H 1400 2000 50  0001 C CNN
+F 2 "Button_Switch_SMD:SW_Push_SPST_NO_Alps_SKRK" H 1400 2000 50  0001 C CNN
 F 3 "~" H 1400 2000 50  0001 C CNN
 	1    1400 1800
@@
 F 0 "SW3" H 2800 4635 50  0000 C CNN
 F 1 "Reset" H 2800 4544 50  0000 C CNN
-F 2 "" H 2800 4550 50  0001 C CNN
+F 2 "Button_Switch_SMD:SW_Push_SPST_NO_Alps_SKRK" H 2800 4550 50  0001 C CNN
 F 3 "~" H 2800 4550 50  0001 C CNN
 	1    2800 4350
@@
 F 0 "SW4" H 3300 6485 50  0000 C CNN
 F 1 "SW_DPDT_x2" H 3300 6394 50  0000 C CNN
-F 2 "" H 3300 6200 50  0001 C CNN
+F 2 "Button_Switch_SMD:SW_SPDT_CK-JS102011SAQN" H 3300 6200 50  0001 C CNN
 F 3 "~" H 3300 6200 50  0001 C CNN
 	1    3300 6200

Commit message: Uso Flag de fuente
Connections:
- net 3.33v: no longer Q1.1 (G), Q2.1 (G)
- net 12v renamed +12V
- net 3.3v renamed +3V3
- net +3V3: now also Q1.1 (G), Q2.1 (G)
- net 5v renamed +5V
Other:
- moved on the sheet: D4, D5, J5, K1, Q4, R14

Commit message: Correccion Esquematico
Parts:
- added R18: 1.8k, symbol Device:R
- added R19: 100k, symbol Device:R
- R14: value 5.6k -> 1.2k
Connections:
- net +3V3: now also C2.1, J2.7 (Pin_7), R1.1, R13.1, SW3.1, U1.2 (VDD)
- net +5V: now also R18.2
- net 3.33v: no longer C2.1, J2.7 (Pin_7), R1.1, R13.1, SW3.1, U1.2 (VDD)
- net GND: now also R19.2; no longer D4.1 (K)
- net at D5.2 (A), K1.2, Q4.1 (C): now also D4.1 (K)
- net at Q4.2 (B), R14.2: now also R19.1; no longer D4.2 (A)
- new net: D4.2 (A), R18.1
- no-connect marks 28 -> 29
Other:
- moved on the sheet: D4

Commit message: Asignacion FootPrint e inicio PCB
Parts:
- C1, C10, C2, C3, C4, C5, C6, C7, C8, C9: footprint (none) -> Capacitor_SMD:C_1210_3225Metric_Pad1.33x2.70mm_HandSolder
- D1, D2, D3, D4, D7, D8: footprint (none) -> LED_SMD:LED_1210_3225Metric_Pad1.42x2.65mm_HandSolder
- F1: footprint (none) -> Fuse:Fuse_1812_4532Metric_Pad1.30x3.40mm_HandSolder
- R1, R10, R11, R12, R13, R14, R15, R16, R17, R18, R19, R2, R3, R4, R5, R6, R7, R8, R9: footprint (none) -> Resistor_SMD:R_0603_1608Metric_Pad0.98x0.95mm_HandSolder
- RV1: footprint (none) -> Potentiometer_THT:Potentiometer_Bourns_3296W_Vertical
Changed lines of the file:
@@
 F 0 "D1" H 3993 2467 50  0000 C CNN
 F 1 "LED" H 3993 2376 50  0000 C CNN
-F 2 "" H 4000 2250 50  0001 C CNN
+F 2 "LED_SMD:LED_1210_3225Metric_Pad1.42x2.65mm_HandSolder" H 4000 2250 50  0001 C CNN
 F 3 "~" H 4000 2250 50  0001 C CNN
 	1    4000 2250
@@
 F 0 "R1" H 870 1846 50  0000 L CNN
 F 1 "10k" H 870 1755 50  0000 L CNN
-F 2 "" V 730 1800 50  0001 C CNN
+F 2 "Resistor_SMD:R_0603_1608Metric_Pad0.98x0.95mm_HandSolder" V 730 1800 50  0001 C CNN
 F 3 "~" H 800 1800 50  0001 C CNN
 	1    800  1800
@@
 F 0 "R2" H 3520 2296 50  0000 L CNN
 F 1 "220" H 3520 2205 50  0000 L CNN
-F 2 "" V 3380 2250 50  0001 C CNN
+F 2 "Resistor_SMD:R_0603_1608Metric_Pad0.98x0.95mm_HandSolder" V 3380 2250 50  0001 C CNN
 F 3 "~" H 3450 2250 50  0001 C CNN
 	1    3450 2250
@@
 F 0 "R13" H 3220 1096 50  0000 L CNN
 F 1 "10k" H 3220 1005 50  0000 L CNN
-F 2 "" V 3080 1050 50  0001 C CNN
+F 2 "Resistor_SMD:R_0603_1608Metric_Pad0.98x0.95mm_HandSolder" V 3080 1050 50  0001 C CNN
 F 3 "~" H 3150 1050 50  0001 C CNN
 	1    3150 1050
@@
 F 0 "R9" H 3320 3046 50  0000 L CNN
 F 1 "10k" H 3320 2955 50  0000 L CNN
-F 2 "" V 3180 3000 50  0001 C CNN
+F 2 "Resistor_SMD:R_0603_1608Metric_Pad0.98x0.95mm_HandSolder" V 3180 3000 50  0001 C CNN
 F 3 "~" H 3250 3000 50  0001 C CNN
 	1    3250 3000
@@
 F 0 "R10" H 3570 3046 50  0000 L CNN
 F 1 "10k" H 3570 2955 50  0000 L CNN
-F 2 "" V 3430 3000 50  0001 C CNN
+F 2 "Resistor_SMD:R_0603_1608Metric_Pad0.98x0.95mm_HandSolder" V 3430 3000 50  0001 C CNN
 F 3 "~" H 3500 3000 50  0001 C CNN
 	1    3500 3000
@@
 F 0 "D2" H 3893 3667 50  0000 C CNN
 F 1 "LED" H 3893 3576 50  0000 C CNN
-F 2 "" H 3900 3450 50  0001 C CNN
+F 2 "LED_SMD:LED_1210_3225Metric_Pad1.42x2.65mm_HandSolder" H 3900 3450 50  0001 C CNN
 F 3 "~" H 3900 3450 50  0001 C CNN
 	1    3900 3450
@@
 F 0 "R11" H 3420 3496 50  0000 L CNN
 F 1 "220" H 3420 3405 50  0000 L CNN
-F 2 "" V 3280 3450 50  0001 C CNN
+F 2 "Resistor_SMD:R_0603_1608Metric_Pad0.98x0.95mm_HandSolder" V 3280 3450 50  0001 C CNN
 F 3 "~" H 3350 3450 50  0001 C CNN
 	1    3350 3450
@@
 F 0 "D3" H 3943 4317 50  0000 C CNN
 F 1 "LED" H 3943 4226 50  0000 C CNN
-F 2 "" H 3950 4100 50  0001 C CNN
+F 2 "LED_SMD:LED_1210_3225Metric_Pad1.42x2.65mm_HandSolder" H 3950 4100 50  0001 C CNN
 F 3 "~" H 3950 4100 50  0001 C CNN
 	1    3950 4100
@@
 F 0 "R12" H 3470 4146 50  0000 L CNN
 F 1 "220" H 3470 4055 50  0000 L CNN
-F 2 "" V 3330 4100 50  0001 C CNN
+F 2 "Resistor_SMD:R_0603_1608Metric_Pad0.98x0.95mm_HandSolder" V 3330 4100 50  0001 C CNN
 F 3 "~" H 3400 4100 50  0001 C CNN
 	1    3400 4100
@@
 F 0 "R14" V 8943 5350 50  0000 C CNN
 F 1 "1.2k" V 9034 5350 50  0000 C CNN
-F 2 "" V 9080 5350 50  0001 C CNN
+F 2 "Resistor_SMD:R_0603_1608Metric_Pad0.98x0.95mm_HandSolder" V 9080 5350 50  0001 C CNN
 F 3 "~" H 9150 5350 50  0001 C CNN
 	1    9150 5350
@@
 F 0 "R8" H 13270 1046 50  0000 L CNN
 F 1 "330" H 13270 955 50  0000 L CNN
-F 2 "" V 13130 1000 50  0001 C CNN
+F 2 "Resistor_SMD:R_0603_1608Metric_Pad0.98x0.95mm_HandSolder" V 13130 1000 50  0001 C CNN
 F 3 "~" H 13200 1000 50  0001 C CNN
 	1    13200 1000
@@
 F 0 "R7" H 8870 2696 50  0000 L CNN
 F 1 "100k" H 8870 2605 50  0000 L CNN
-F 2 "" V 8730 2650 50  0001 C CNN
+F 2 "Resistor_SMD:R_0603_1608Metric_Pad0.98x0.95mm_HandSolder" V 8730 2650 50  0001 C CNN
 F 3 "~" H 8800 2650 50  0001 C CNN
 	1    8800 2650
@@
 F 0 "R6" H 8870 2396 50  0000 L CNN
 F 1 "100k" H 8870 2305 50  0000 L CNN
-F 2 "" V 8730 2350 50  0001 C CNN
+F 2 "Resistor_SMD:R_0603_1608Metric_Pad0.98x0.95mm_HandSolder" V 8730 2350 50  0001 C CNN
 F 3 "~" H 8800 2350 50  0001 C CNN
 	1    8800 2350
@@
 F 0 "R5" H 8870 2096 50  0000 L CNN
 F 1 "100k" H 8870 2005 50  0000 L CNN
-F 2 "" V 8730 2050 50  0001 C CNN
+F 2 "Resistor_SMD:R_0603_1608Metric_Pad0.98x0.95mm_HandSolder" V 8730 2050 50  0001 C CNN
 F 3 "~" H 8800 2050 50  0001 C CNN
 	1    8800 2050
@@
 F 0 "R4" H 8320 1196 50  0000 L CNN
 F 1 "10k" H 8320 1105 50  0000 L CNN
-F 2 "" V 8180 1150 50  0001 C CNN
+F 2 "Resistor_SMD:R_0603_1608Metric_Pad0.98x0.95mm_HandSolder" V 8180 1150 50  0001 C CNN
 F 3 "~" H 8250 1150 50  0001 C CNN
 	1    8250 1150
@@
 F 0 "R3" H 8070 1196 50  0000 L CNN
 F 1 "10k" H 8070 1105 50  0000 L CNN
-F 2 "" V 7930 1150 50  0001 C CNN
+F 2 "Resistor_SMD:R_0603_1608Metric_Pad0.98x0.95mm_HandSolder" V 7930 1150 50  0001 C CNN
 F 3 "~" H 8000 1150 50  0001 C CNN
 	1    8000 1150
@@
 F 0 "RV1" H 10530 1096 50  0000 R CNN
 F 1 "10k" H 10530 1005 50  0000 R CNN
-F 2 "" H 10600 1050 50  0001 C CNN
+F 2 "Potentiometer_THT:Potentiometer_Bourns_3296W_Vertical" H 10600 1050 50  0001 C CNN
 F 3 "~" H 10600 1050 50  0001 C CNN
 	1    10600 1050
@@
 F 0 "R15" H 2370 6496 50  0000 L CNN
 F 1 "100k" H 2370 6405 50  0000 L CNN
-F 2 "" V 2230 6450 50  0001 C CNN
+F 2 "Resistor_SMD:R_0603_1608Metric_Pad0.98x0.95mm_HandSolder" V 2230 6450 50  0001 C CNN
 F 3 "~" H 2300 6450 50  0001 C CNN
 	1    2300 6450
@@
 F 0 "F1" H 1460 6246 50  0000 L CNN
 F 1 "Fuse" H 1460 6155 50  0000 L CNN
-F 2 "" V 1330 6200 50  0001 C CNN
+F 2 "Fuse:Fuse_1812_4532Metric_Pad1.30x3.40mm_HandSolder" V 1330 6200 50  0001 C CNN
 F 3 "~" H 1400 6200 50  0001 C CNN
 	1    1400 6200
@@
 F 0 "C10" H 7865 6546 50  0000 L CNN
 F 1 "100n" H 7865 6455 50  0000 L CNN
-F 2 "" H 7788 6350 50  0001 C CNN
+F 2 "Capacitor_SMD:C_1210_3225Metric_Pad1.33x2.70mm_HandSolder" H 7788 6350 50  0001 C CNN
 F 3 "~" H 7750 6500 50  0001 C CNN
 	1    7750 6500
@@
 F 0 "C9" H 7515 6546 50  0000 L CNN
 F 1 "22u" H 7515 6455 50  0000 L CNN
-F 2 "" H 7400 6500 50  0001 C CNN
+F 2 "Capacitor_SMD:C_1210_3225Metric_Pad1.33x2.70mm_HandSolder" H 7400 6500 50  0001 C CNN
 F 3 "~" H 7400 6500 50  0001 C CNN
 	1    7400 6500
@@
 F 0 "C8" H 6415 6546 50  0000 L CNN
 F 1 "100n" H 6415 6455 50  0000 L CNN
-F 2 "" H 6338 6350 50  0001 C CNN
+F 2 "Capacitor_SMD:C_1210_3225Metric_Pad1.33x2.70mm_HandSolder" H 6338 6350 50  0001 C CNN
 F 3 "~" H 6300 6500 50  0001 C CNN
 	1    6300 6500
@@
 F 0 "C7" H 6065 6546 50  0000 L CNN
 F 1 "22u" H 6065 6455 50  0000 L CNN
-F 2 "" H 5950 6500 50  0001 C CNN
+F 2 "Capacitor_SMD:C_1210_3225Metric_Pad1.33x2.70mm_HandSolder" H 5950 6500 50  0001 C CNN
 F 3 "~" H 5950 6500 50  0001 C CNN
 	1    5950 6500
@@
 F 0 "C4" H 4265 6546 50  0000 L CNN
 F 1 "100n" H 4265 6455 50  0000 L CNN
-F 2 "" H 4188 6350 50  0001 C CNN
+F 2 "Capacitor_SMD:C_1210_3225Metric_Pad1.33x2.70mm_HandSolder" H 4188 6350 50  0001 C CNN
 F 3 "~" H 4150 6500 50  0001 C CNN
 	1    4150 6500
@@
 F 0 "C6" H 5565 6546 50  0000 L CNN
 F 1 "100u" H 5565 6455 50  0000 L CNN
-F 2 "" H 5450 6500 50  0001 C CNN
+F 2 "Capacitor_SMD:C_1210_3225Metric_Pad1.33x2.70mm_HandSolder" H 5450 6500 50  0001 C CNN
 F 3 "~" H 5450 6500 50  0001 C CNN
 	1    5450 6500
@@
 F 0 "C5" H 4665 6546 50  0000 L CNN
 F 1 "100u" H 4665 6455 50  0000 L CNN
-F 2 "" H 4550 6500 50  0001 C CNN
+F 2 "Capacitor_SMD:C_1210_3225Metric_Pad1.33x2.70mm_HandSolder" H 4550 6500 50  0001 C CNN
 F 3 "~" H 4550 6500 50  0001 C CNN
 	1    4550 6500
@@
 F 0 "C2" V 3052 4600 50  0000 C CNN
 F 1 "10u" V 2961 4600 50  0000 C CNN
-F 2 "" H 2838 4450 50  0001 C CNN
+F 2 "Capacitor_SMD:C_1210_3225Metric_Pad1.33x2.70mm_HandSolder" H 2838 4450 50  0001 C CNN
 F 3 "~" H 2800 4600 50  0001 C CNN
 	1    2800 4600
@@
 F 0 "C1" V 1652 2050 50  0000 C CNN
 F 1 "10u" V 1561 2050 50  0000 C CNN
-F 2 "" H 1438 1900 50  0001 C CNN
+F 2 "Capacitor_SMD:C_1210_3225Metric_Pad1.33x2.70mm_HandSolder" H 1438 1900 50  0001 C CNN
 F 3 "~" H 1400 2050 50  0001 C CNN
 	1    1400 2050
@@
 F 0 "C3" V 4302 800 50  0000 C CNN
 F 1 "10u" V 4211 800 50  0000 C CNN
-F 2 "" H 4088 650 50  0001 C CNN
+F 2 "Capacitor_SMD:C_1210_3225Metric_Pad1.33x2.70mm_HandSolder" H 4088 650 50  0001 C CNN
 F 3 "~" H 4050 800 50  0001 C CNN
 	1    4050 800
@@
 F 0 "R17" H 3770 6496 50  0000 L CNN
 F 1 "1k" H 3770 6405 50  0000 L CNN
-F 2 "" V 3630 6450 50  0001 C CNN
+F 2 "Resistor_SMD:R_0603_1608Metric_Pad0.98x0.95mm_HandSolder" V 3630 6450 50  0001 C CNN
 F 3 "~" H 3700 6450 50  0001 C CNN
 	1    3700 6450
@@
 F 0 "R16" H 1870 6546 50  0000 L CNN
 F 1 "1k" H 1870 6455 50  0000 L CNN
-F 2 "" V 1730 6500 50  0001 C CNN
+F 2 "Resistor_SMD:R_0603_1608Metric_Pad0.98x0.95mm_HandSolder" V 1730 6500 50  0001 C CNN
 F 3 "~" H 1800 6500 50  0001 C CNN
 	1    1800 6500
@@
 F 0 "D8" H 3693 7167 50  0000 C CNN
 F 1 "LED" H 3693 7076 50  0000 C CNN
-F 2 "" H 3700 6950 50  0001 C CNN
+F 2 "LED_SMD:LED_1210_3225Metric_Pad1.42x2.65mm_HandSolder" H 3700 6950 50  0001 C CNN
 F 3 "~" H 3700 6950 50  0001 C CNN
 	1    3700 6950
@@
 F 0 "D7" H 1793 7167 50  0000 C CNN
 F 1 "LED" H 1793 7076 50  0000 C CNN
-F 2 "" H 1800 6950 50  0001 C CNN
+F 2 "LED_SMD:LED_1210_3225Metric_Pad1.42x2.65mm_HandSolder" H 1800 6950 50  0001 C CNN
 F 3 "~" H 1800 6950 50  0001 C CNN
 	1    1800 6950
@@
 F 0 "D4" H 8743 5067 50  0000 C CNN
 F 1 "LED" H 8743 4976 50  0000 C CNN
-F 2 "" H 8750 4850 50  0001 C CNN
+F 2 "LED_SMD:LED_1210_3225Metric_Pad1.42x2.65mm_HandSolder" H 8750 4850 50  0001 C CNN
 F 3 "~" H 8750 4850 50  0001 C CNN
 	1    8750 4850
@@
 F 0 "R19" H 9570 5996 50  0000 L CNN
 F 1 "100k" H 9570 5905 50  0000 L CNN
-F 2 "" V 9430 5950 50  0001 C CNN
+F 2 "Resistor_SMD:R_0603_1608Metric_Pad0.98x0.95mm_HandSolder" V 9430 5950 50  0001 C CNN
 F 3 "~" H 9500 5950 50  0001 C CNN
 	1    9500 5950
@@
 F 0 "R18" V 9207 4400 50  0000 C CNN
 F 1 "1.8k" V 9116 4400 50  0000 C CNN
-F 2 "" V 8930 4400 50  0001 C CNN
+F 2 "Resistor_SMD:R_0603_1608Metric_Pad0.98x0.95mm_HandSolder" V 8930 4400 50  0001 C CNN
 F 3 "~" H 9000 4400 50  0001 C CNN
 	1    9000 4400

Commit message: D
Parts:
- U2, U3: footprint Display:NHD-0420H1Z -> Display:WC1602A
Changed lines of the file:
@@
 F 0 "U2" H 12550 561 50  0000 C CNN
 F 1 "NHD-0420H1Z" H 12550 470 50  0000 C CNN
-F 2 "Display:NHD-0420H1Z" H 12550 550 50  0001 C CNN
+F 2 "Display:WC1602A" H 12550 550 50  0001 C CNN
 F 3 "http://www.newhavendisplay.com/specs/NHD-0420H1Z-FSW-GBW-33V3.pdf" H 12650 1350 50  0001 C CNN
 	1    12550 1450
@@
 F 0 "U3" H 12550 2511 50  0000 C CNN
 F 1 "NHD-0420H1Z" H 12550 2420 50  0000 C CNN
-F 2 "Display:NHD-0420H1Z" H 12550 2500 50  0001 C CNN
+F 2 "Display:WC1602A" H 12550 2500 50  0001 C CNN
 F 3 "http://www.newhavendisplay.com/specs/NHD-0420H1Z-FSW-GBW-33V3.pdf" H 12650 3300 50  0001 C CNN
 	1    12550 3400

Commit message: Inicio PCB
Parts:
- U2, U3: footprint Display:WC1602A -> LIB:LCD_LCD-20X4B
Connections:
- net 3.33v is gone; now on net +3V3: R10.2, R9.2
- net MISO: no longer names the net of J2.4 (Pin_4), U1.31 (IO19)
- net MOSI: no longer names the net of J2.3 (Pin_3), U1.37 (IO23)
- net RST: no longer names the net of J2.6 (Pin_6), U1.28 (IO17)
- net SCKs: no longer names the net of J2.2 (Pin_2), U1.16 (IO13)
- net SDAs: no longer names the net of J2.1 (Pin_1), U1.29 (IO5)
Changed lines of the file:
@@
 Wire Wire Line
 	3250 3150 3400 3150
-Text GLabel 3550 3250 2    50   Input ~ 0
-3.33v
 Wire Wire Line
 	3400 3150 3400 3250
-Wire Wire Line
-	3400 3250 3550 3250
 Connection ~ 3400 3150
 Wire Wire Line
@@
 Wire Wire Line
 	3800 4100 3550 4100
-Text GLabel 4450 2350 3    50   Input ~ 0
-RST
 Wire Wire Line
 	2400 1050 3000 1050
@@
 Wire Wire Line
 	3750 750  3750 2450
-Text GLabel 4700 1800 0    50   Input ~ 0
-SDAs
-Text GLabel 3600 1950 1    50   Input ~ 0
-SCKs
 $Comp
 L Connector:Conn_01x07_Female J2
@@
 Wire Wire Line
 	3100 2850 3000 2850
-Text GLabel 3200 2050 3    50   Input ~ 0
-MOSI
 Wire Wire Line
 	3000 2550 4650 2550
@@
 Wire Wire Line
 	4650 2150 4800 2150
-Text GLabel 4650 2550 3    50   Input ~ 0
-MISO
 Wire Wire Line
 	4050 3450 4350 3450
@@
 F 0 "U2" H 12550 561 50  0000 C CNN
 F 1 "NHD-0420H1Z" H 12550 470 50  0000 C CNN
-F 2 "Display:WC1602A" H 12550 550 50  0001 C CNN
+F 2 "LIB:LCD_LCD-20X4B" H 12550 550 50  0001 C CNN
 F 3 "http://www.newhavendisplay.com/specs/NHD-0420H1Z-FSW-GBW-33V3.pdf" H 12650 1350 50  0001 C CNN
 	1    12550 1450
@@
 Wire Wire Line
 	4550 6200 4150 6200
-Connection ~ 4150 6200
 Wire Wire Line
 	4150 6350 4150 6200
@@
 Wire Wire Line
 	3700 6300 3700 6200
-Connection ~ 3700 6200
 Wire Wire Line
 	3700 6600 3700 6800
@@
 L power:+12V #PWR0110
 U 1 1 62FAF0A2
-P 4000 6150
-F 0 "#PWR0110" H 4000 6000 50  0001 C CNN
-F 1 "+12V" H 4015 6323 50  0000 C CNN
-F 2 "" H 4000 6150 50  0001 C CNN
-F 3 "" H 4000 6150 50  0001 C CNN
-	1    4000 6150
+P 3950 6000
+F 0 "#PWR0110" H 3950 5850 50  0001 C CNN
+F 1 "+12V" H 3965 6173 50  0000 C CNN
+F 2 "" H 3950 6000 50  0001 C CNN
+F 3 "" H 3950 6000 50  0001 C CNN
+	1    3950 6000
 	1    0    0    -1
 $EndComp
@@
 F 0 "U3" H 12550 2511 50  0000 C CNN
 F 1 "NHD-0420H1Z" H 12550 2420 50  0000 C CNN
-F 2 "Display:WC1602A" H 12550 2500 50  0001 C CNN
+F 2 "LIB:LCD_LCD-20X4B" H 12550 2500 50  0001 C CNN
 F 3 "http://www.newhavendisplay.com/specs/NHD-0420H1Z-FSW-GBW-33V3.pdf" H 12650 3300 50  0001 C CNN
 	1    12550 3400
@@
 Wire Wire Line
 	10400 2550 12650 2550
-Wire Wire Line
-	3700 6200 4000 6200
-Wire Wire Line
-	4000 6150 4000 6200
-Connection ~ 4000 6200
-Wire Wire Line
-	4000 6200 4150 6200
 Wire Wire Line
 	8650 3850 8650 3950
@@
 	10450 600  12650 600
 Connection ~ 10450 1050
+$Comp
+L power:+3.3V #PWR0114
+U 1 1 629515F0
+P 4900 3200
+F 0 "#PWR0114" H 4900 3050 50  0001 C CNN
+F 1 "+3.3V" H 4915 3373 50  0000 C CNN
+F 2 "" H 4900 3200 50  0001 C CNN
+F 3 "" H 4900 3200 50  0001 C CNN
+	1    4900 3200
+	1    0    0    -1
+$EndComp
+Wire Wire Line
+	4900 3250 4900 3200
+Wire Wire Line
+	3400 3250 4900 3250
+Wire Wire Line
+	4150 6200 3950 6200
+Connection ~ 4150 6200
+Connection ~ 3700 6200
+Wire Wire Line
+	3950 6000 3950 6200
+Connection ~ 3950 6200
+Wire Wire Line
+	3950 6200 3700 6200
 $EndSCHEMATC

Commit message: Distribucion final de componetes en 10*10
Parts:
- SW1: value SW_Push -> Program
Changed lines of the file:
@@
 P 4050 1250
 F 0 "SW1" H 4050 1535 50  0000 C CNN
-F 1 "SW_Push" H 4050 1444 50  0000 C CNN
+F 1 "Program" H 4050 1444 50  0000 C CNN
 F 2 "Button_Switch_SMD:SW_Push_SPST_NO_Alps_SKRK" H 4050 1450 50  0001 C CNN
 F 3 "~" H 4050 1450 50  0001 C CNN

Commit message: Ajustes Finales PCB
Parts:
- C1, C10, C2, C3, C4, C5, C6, C7, C8, C9: footprint Capacitor_SMD:C_1210_3225Metric_Pad1.33x2.70mm_HandSolder -> Capacitor_SMD:C_1206_3216Metric_Pad1.33x1.80mm_HandSolder
- D1, D2, D3, D4, D7, D8: footprint LED_SMD:LED_1210_3225Metric_Pad1.42x2.65mm_HandSolder -> LED_SMD:LED_0805_2012Metric_Pad1.15x1.40mm_HandSolder
Changed lines of the file:
@@
 F 0 "D1" H 3993 2467 50  0000 C CNN
 F 1 "LED" H 3993 2376 50  0000 C CNN
-F 2 "LED_SMD:LED_1210_3225Metric_Pad1.42x2.65mm_HandSolder" H 4000 2250 50  0001 C CNN
+F 2 "LED_SMD:LED_0805_2012Metric_Pad1.15x1.40mm_HandSolder" H 4000 2250 50  0001 C CNN
 F 3 "~" H 4000 2250 50  0001 C CNN
 	1    4000 2250
@@
 F 0 "D2" H 3893 3667 50  0000 C CNN
 F 1 "LED" H 3893 3576 50  0000 C CNN
-F 2 "LED_SMD:LED_1210_3225Metric_Pad1.42x2.65mm_HandSolder" H 3900 3450 50  0001 C CNN
+F 2 "LED_SMD:LED_0805_2012Metric_Pad1.15x1.40mm_HandSolder" H 3900 3450 50  0001 C CNN
 F 3 "~" H 3900 3450 50  0001 C CNN
 	1    3900 3450
@@
 F 0 "D3" H 3943 4317 50  0000 C CNN
 F 1 "LED" H 3943 4226 50  0000 C CNN
-F 2 "LED_SMD:LED_1210_3225Metric_Pad1.42x2.65mm_HandSolder" H 3950 4100 50  0001 C CNN
+F 2 "LED_SMD:LED_0805_2012Metric_Pad1.15x1.40mm_HandSolder" H 3950 4100 50  0001 C CNN
 F 3 "~" H 3950 4100 50  0001 C CNN
 	1    3950 4100
@@
 F 0 "C10" H 7865 6546 50  0000 L CNN
 F 1 "100n" H 7865 6455 50  0000 L CNN
-F 2 "Capacitor_SMD:C_1210_3225Metric_Pad1.33x2.70mm_HandSolder" H 7788 6350 50  0001 C CNN
+F 2 "Capacitor_SMD:C_1206_3216Metric_Pad1.33x1.80mm_HandSolder" H 7788 6350 50  0001 C CNN
 F 3 "~" H 7750 6500 50  0001 C CNN
 	1    7750 6500
@@
 F 0 "C9" H 7515 6546 50  0000 L CNN
 F 1 "22u" H 7515 6455 50  0000 L CNN
-F 2 "Capacitor_SMD:C_1210_3225Metric_Pad1.33x2.70mm_HandSolder" H 7400 6500 50  0001 C CNN
+F 2 "Capacitor_SMD:C_1206_3216Metric_Pad1.33x1.80mm_HandSolder" H 7400 6500 50  0001 C CNN
 F 3 "~" H 7400 6500 50  0001 C CNN
 	1    7400 6500
@@
 F 0 "C8" H 6415 6546 50  0000 L CNN
 F 1 "100n" H 6415 6455 50  0000 L CNN
-F 2 "Capacitor_SMD:C_1210_3225Metric_Pad1.33x2.70mm_HandSolder" H 6338 6350 50  0001 C CNN
+F 2 "Capacitor_SMD:C_1206_3216Metric_Pad1.33x1.80mm_HandSolder" H 6338 6350 50  0001 C CNN
 F 3 "~" H 6300 6500 50  0001 C CNN
 	1    6300 6500
@@
 F 0 "C7" H 6065 6546 50  0000 L CNN
 F 1 "22u" H 6065 6455 50  0000 L CNN
-F 2 "Capacitor_SMD:C_1210_3225Metric_Pad1.33x2.70mm_HandSolder" H 5950 6500 50  0001 C CNN
+F 2 "Capacitor_SMD:C_1206_3216Metric_Pad1.33x1.80mm_HandSolder" H 5950 6500 50  0001 C CNN
 F 3 "~" H 5950 6500 50  0001 C CNN
 	1    5950 6500
@@
 F 0 "C4" H 4265 6546 50  0000 L CNN
 F 1 "100n" H 4265 6455 50  0000 L CNN
-F 2 "Capacitor_SMD:C_1210_3225Metric_Pad1.33x2.70mm_HandSolder" H 4188 6350 50  0001 C CNN
+F 2 "Capacitor_SMD:C_1206_3216Metric_Pad1.33x1.80mm_HandSolder" H 4188 6350 50  0001 C CNN
 F 3 "~" H 4150 6500 50  0001 C CNN
 	1    4150 6500
@@
 F 0 "C6" H 5565 6546 50  0000 L CNN
 F 1 "100u" H 5565 6455 50  0000 L CNN
-F 2 "Capacitor_SMD:C_1210_3225Metric_Pad1.33x2.70mm_HandSolder" H 5450 6500 50  0001 C CNN
+F 2 "Capacitor_SMD:C_1206_3216Metric_Pad1.33x1.80mm_HandSolder" H 5450 6500 50  0001 C CNN
 F 3 "~" H 5450 6500 50  0001 C CNN
 	1    5450 6500
@@
 F 0 "C5" H 4665 6546 50  0000 L CNN
 F 1 "100u" H 4665 6455 50  0000 L CNN
-F 2 "Capacitor_SMD:C_1210_3225Metric_Pad1.33x2.70mm_HandSolder" H 4550 6500 50  0001 C CNN
+F 2 "Capacitor_SMD:C_1206_3216Metric_Pad1.33x1.80mm_HandSolder" H 4550 6500 50  0001 C CNN
 F 3 "~" H 4550 6500 50  0001 C CNN
 	1    4550 6500
@@
 F 0 "C2" V 3052 4600 50  0000 C CNN
 F 1 "10u" V 2961 4600 50  0000 C CNN
-F 2 "Capacitor_SMD:C_1210_3225Metric_Pad1.33x2.70mm_HandSolder" H 2838 4450 50  0001 C CNN
+F 2 "Capacitor_SMD:C_1206_3216Metric_Pad1.33x1.80mm_HandSolder" H 2838 4450 50  0001 C CNN
 F 3 "~" H 2800 4600 50  0001 C CNN
 	1    2800 4600
@@
 F 0 "C1" V 1652 2050 50  0000 C CNN
 F 1 "10u" V 1561 2050 50  0000 C CNN
-F 2 "Capacitor_SMD:C_1210_3225Metric_Pad1.33x2.70mm_HandSolder" H 1438 1900 50  0001 C CNN
+F 2 "Capacitor_SMD:C_1206_3216Metric_Pad1.33x1.80mm_HandSolder" H 1438 1900 50  0001 C CNN
 F 3 "~" H 1400 2050 50  0001 C CNN
 	1    1400 2050
@@
 F 0 "C3" V 4302 800 50  0000 C CNN
 F 1 "10u" V 4211 800 50  0000 C CNN
-F 2 "Capacitor_SMD:C_1210_3225Metric_Pad1.33x2.70mm_HandSolder" H 4088 650 50  0001 C CNN
+F 2 "Capacitor_SMD:C_1206_3216Metric_Pad1.33x1.80mm_HandSolder" H 4088 650 50  0001 C CNN
 F 3 "~" H 4050 800 50  0001 C CNN
 	1    4050 800
@@
 F 0 "D8" H 3693 7167 50  0000 C CNN
 F 1 "LED" H 3693 7076 50  0000 C CNN
-F 2 "LED_SMD:LED_1210_3225Metric_Pad1.42x2.65mm_HandSolder" H 3700 6950 50  0001 C CNN
+F 2 "LED_SMD:LED_0805_2012Metric_Pad1.15x1.40mm_HandSolder" H 3700 6950 50  0001 C CNN
 F 3 "~" H 3700 6950 50  0001 C CNN
 	1    3700 6950
@@
 F 0 "D7" H 1793 7167 50  0000 C CNN
 F 1 "LED" H 1793 7076 50  0000 C CNN
-F 2 "LED_SMD:LED_1210_3225Metric_Pad1.42x2.65mm_HandSolder" H 1800 6950 50  0001 C CNN
+F 2 "LED_SMD:LED_0805_2012Metric_Pad1.15x1.40mm_HandSolder" H 1800 6950 50  0001 C CNN
 F 3 "~" H 1800 6950 50  0001 C CNN
 	1    1800 6950
@@
 F 0 "D4" H 8743 5067 50  0000 C CNN
 F 1 "LED" H 8743 4976 50  0000 C CNN
-F 2 "LED_SMD:LED_1210_3225Metric_Pad1.42x2.65mm_HandSolder" H 8750 4850 50  0001 C CNN
+F 2 "LED_SMD:LED_0805_2012Metric_Pad1.15x1.40mm_HandSolder" H 8750 4850 50  0001 C CNN
 F 3 "~" H 8750 4850 50  0001 C CNN
 	1    8750 4850
